File: schematics/schematics/eMH1/eMH1.sch (KiCad schematic (older format))
At the start: 9 parts, among them IC1 DIL14, IC2 DIL20, K1 CONN_3, P1 CONN_5X2, P2 USB

Commit message: eMH1 continued
Connections:
- net GND: now also IC1.14
- net at IC2.1 (P1), P2.1 (Vbus), R?.1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: now also IC1.1
- net at IC2.10 (P10): now also IC1.5
- net at IC2.12 (P12): now also IC1.6
Changed lines of the file:
@@
-EESchema Schematic File Version 2  date 2012. 02. 24. 19:55:58
+EESchema Schematic File Version 2  date 2012. febr. 25., szombat, 18.37.38 CET
 LIBS:power
 LIBS:device
@@
 LIBS:contrib
 LIBS:valves
-EELAYER 43  0
+EELAYER 25  0
 EELAYER END
-$Descr A4 11700 8267
+$Descr A4 11693 8268
 encoding utf-8
 Sheet 1 1
 Title ""
-Date "24 feb 2012"
+Date "25 feb 2012"
 Rev ""
 Comp ""
@@
 Comment4 ""
 $EndDescr
-NoConn ~ 1400 3650
-NoConn ~ 2150 3650
-Connection ~ 2100 4600
 Wire Wire Line
-	2100 4600 3300 4600
+	7100 4100 5600 4100
 Wire Wire Line
-	3300 4600 3300 4150
+	5600 4100 5600 4750
 Wire Wire Line
-	3300 4150 3150 4150
+	5600 4750 4550 4750
+Connection ~ 1300 3400
 Wire Wire Line
-	1650 5100 1650 5200
+	1300 3400 1300 2650
 Wire Wire Line
-	1650 5200 2900 5200
+	1300 2650 5500 2650
 Wire Wire Line
-	2900 5200 2900 4350
+	5500 2650 5500 3600
 Wire Wire Line
-	2900 4350 3850 4350
+	5500 3600 7100 3600
 Wire Wire Line
-	1350 4700 1350 4600
-Connection ~ 1350 3950
+	1350 5100 1350 5250
 Wire Wire Line
-	1350 4100 1350 3950
+	1350 5250 2950 5250
 Wire Wire Line
-	4550 4150 4700 4150
+	2950 5250 2950 4450
 Wire Wire Line
-	4700 4150 4700 3550
+	2950 4450 3850 4450
 Wire Wire Line
-	4700 3550 2150 3550
+	1650 4700 1650 4600
+Connection ~ 1650 3950
 Wire Wire Line
-	1400 3550 1200 3550
+	1650 4100 1650 3950
+Connection ~ 2100 3850
 Wire Wire Line
-	1200 3550 1200 3850
+	2100 3850 2100 5450
 Wire Wire Line
-	1200 3850 3600 3850
+	2150 3400 4600 3400
 Wire Wire Line
-	3600 3850 3600 3750
+	4600 3400 4600 4050
 Wire Wire Line
-	3600 3750 4550 3750
+	4600 4050 4550 4050
 Wire Wire Line
-	4550 3750 4550 3950
+	1400 3400 1100 3400
 Wire Wire Line
-	3150 4250 3400 4250
+	1100 3400 1100 3950
 Wire Wire Line
-	3400 4250 3400 4150
-Wire Wire Line
-	3400 4150 3850 4150
+	1100 3950 3850 3950
 Wire Wire Line
 	3850 4050 3150 4050
 Wire Wire Line
-	3850 3950 1100 3950
+	3850 4150 3400 4150
 Wire Wire Line
-	1100 3950 1100 3400
+	3400 4150 3400 4250
 Wire Wire Line
-	1100 3400 1400 3400
+	3400 4250 3150 4250
 Wire Wire Line
-	4550 4050 4600 4050
+	4550 3950 4550 3750
 Wire Wire Line
-	4600 4050 4600 3400
+	4550 3750 3600 3750
 Wire Wire Line
-	4600 3400 2150 3400
+	3600 3750 3600 3850
 Wire Wire Line
-	2100 5450 2100 3850
-Connection ~ 2100 3850
+	3600 3850 1200 3850
 Wire Wire Line
-	1650 4100 1650 3950
-Connection ~ 1650 3950
+	1200 3550 1400 3550
 Wire Wire Line
-	1650 4700 1650 4600
+	2150 3550 4700 3550
 Wire Wire Line
-	3850 4450 2950 4450
+	4700 3550 4700 4150
 Wire Wire Line
-	2950 4450 2950 5250
+	4700 4150 4550 4150
 Wire Wire Line
-	2950 5250 1350 5250
+	1350 3950 1350 4100
+Connection ~ 1350 3950
 Wire Wire Line
-	1350 5250 1350 5100
+	1350 4700 1350 4600
+Wire Wire Line
+	3850 4350 2900 4350
+Wire Wire Line
+	2900 4350 2900 5200
+Wire Wire Line
+	2900 5200 1650 5200
+Wire Wire Line
+	1650 5200 1650 5100
+Wire Wire Line
+	3150 4150 3300 4150
+Wire Wire Line
+	3300 4150 3300 4600
+Wire Wire Line
+	3300 4600 2100 4600
+Connection ~ 2100 4600
+Wire Wire Line
+	1200 3850 1200 2600
+Wire Wire Line
+	1200 2600 6400 2600
+Wire Wire Line
+	6400 2600 6400 3400
+Wire Wire Line
+	6400 3400 7900 3400
+Wire Wire Line
+	7900 3400 7900 3600
+Wire Wire Line
+	7900 3600 7800 3600
+Connection ~ 1200 3550
+Wire Wire Line
+	3850 4850 3700 4850
+Wire Wire Line
+	3700 4850 3700 5000
+Wire Wire Line
+	3700 5000 5500 5000
+Wire Wire Line
+	5500 5000 5500 4000
+Wire Wire Line
+	5500 4000 7100 4000
+NoConn ~ 1400 3650
+NoConn ~ 2150 3650
 $Comp
 L R R?

Commit message: eMH1 continued
Parts:
- added P3: CONN_6, symbol CONN_6
- added R? (x3): R, symbol R
Connections:
- net GND: now also P1.2, P3.3
- net at IC1.1, IC2.1 (P1), P2.1 (Vbus)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: now also P1.1, P3.2, R?.1, R?.1, R?.1
- net at IC2.11 (P11): now also IC1.3
- net at IC2.13 (P13): now also IC1.2
- net at IC2.16 (P16): now also IC1.11
- net at IC2.4 (P4): now also R?.2
- net at IC2.8 (P8): now also P1.9
- net at IC2.9 (P9): now also P1.7
- net at IC1.10: now also P1.3, R?.2
- net at IC1.12: now also P3.5
- net at IC1.13: now also P3.4
- net at IC1.4: now also P3.1
- net at IC1.7: now also P1.5
- net at IC1.8: now also P1.6
- net at IC1.9: now also P1.4, R?.2
- no-connect marks 2 -> 5
Other:
- note added: "P2 Connector:\n1- Vdd\n2- Vss\n3- I2C clock SCL\n4- I2C data SDA\n5- Trigger1\n6- Trigger2\n7- Trigger3\n8- NC\n9- Trigger4\n10- NC"
- moved on the sheet: P1
