File: schematics/eMP1/eMP1.sch (KiCad schematic (older format))
At the start: 31 parts, among them IC1 MCP2200, IC2 PIC16F1824, IC3 PIC16F1824, IC4 L298, J1 USB_2, J2 JUMPER, P1 CONN_6, P10 CONN_4, P11 CONN_4, P2 CONN_6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

Commit message: eMP1 gerber and PDF plot
Parts:
- removed C2: CP1, symbol CP1
- added C2: CP, symbol CP
Connections:
- net at IC1.1 (Vdd), J1.1, R1.2: now also C2.1
- net at C1.1, IC1.20 (Vss), J1.4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: now also C2.2
Changed lines of the file:
@@
-EESchema Schematic File Version 2  date Thu 15 Mar 2012 14:03:59 CET
+EESchema Schematic File Version 2  date 2012. 03. 22. 18:04:01
 LIBS:resonator
 LIBS:power
@@
 LIBS:mcp2200
 LIBS:pic16f1824
-EELAYER 43  0
+LIBS:eMP1-cache
+EELAYER 25  0
 EELAYER END
 $Descr A4 11700 8267
@@
 Sheet 1 1
 Title ""
-Date "15 mar 2012"
+Date "22 mar 2012"
 Rev ""
 Comp ""
@@
 Comment4 ""
 $EndDescr
+$Comp
+L CP C2
+U 1 1 4F6B5ADD
+P 3550 1500
+F 0 "C2" H 3600 1600 50  0000 L CNN
+F 1 "CP" H 3600 1400 50  0000 L CNN
+	1    3550 1500
+	0    -1   -1   0
+$EndComp
 Wire Wire Line
 	5050 4900 3950 4900
@@
 $EndComp
 $Comp
-L CP1 C2
-U 1 1 4F61DD2E
-P 3550 1500
-F 0 "C2" H 3600 1600 50  0000 L CNN
-F 1 "CP1" H 3600 1400 50  0000 L CNN
-	1    3550 1500
-	0    -1   1    0
-$EndComp
-$Comp
